File: pcb/main/main.sch (KiCad schematic (older format))
At the start: 42 parts, among them J1 USB_B_Micro, J2 Conn_01x12, J3 ISP, J4 Conn_01x12, Q1 FDN340P, SW1 SW_Push, U1 CH340G, U2 TLV70033, U3 ATmega328P-AU, U4 RFM95W-915S2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

Commit message: Minor fixes in schematic
Connections:
- wire segments 216 -> 220
Other:
- moved on the sheet: BT1, C6, C7, D1, R1, R4, R5, U2

Commit message: Added DNP for antenna matching components values
Parts:
- C17, C18: value C -> DNP
- D2: value LED -> LED_Y
- L1: value L -> DNP
Other:
- moved on the sheet: D2, J2, J3, J4, R6, R7, SW1

Commit message: Footprints assigned
Parts:
- removed AE1: PCB_F_ANTENNA, symbol Device:Antenna_Shield
- removed D1: MBR0540, Diode_SMD:D_SOD-123, symbol Diode:MBR0540
- removed Q1: FDN340P, Package_TO_SOT_SMD:SOT-23, symbol Transistor_FET:FDN340P
- added D1: MBR0520, Diode_SMD:D_SOD-123, symbol Diode:MBR0520
- added Q1: DMP3099L, Package_TO_SOT_SMD:SOT-23, symbol Transistor_FET:DMP3099L
- BT1: footprint (none) -> Battery:BatteryHolder_MPD_BH-18650-PC2
- C1, C10, C11, C12, C13, C14, C15, C16, C17, C18, C2, C3, C5, C7, C8, C9: footprint (none) -> Capacitor_SMD:C_0805_2012Metric_Pad1.18x1.45mm_HandSolder
- C4, C6: value 0.1uF -> 100nF; footprint (none) -> Capacitor_SMD:C_0805_2012Metric_Pad1.18x1.45mm_HandSolder
- D2: footprint (none) -> LED_SMD:LED_0805_2012Metric_Pad1.15x1.40mm_HandSolder
- J1: footprint (none) -> Connector_USB:USB_Micro-B_Molex_47346-0001
- J2, J4: footprint (none) -> Connector_PinHeader_2.54mm:PinHeader_1x12_P2.54mm_Vertical
- J3: footprint (none) -> Connector_PinHeader_2.54mm:PinHeader_2x03_P2.54mm_Vertical
- L1: footprint (none) -> Inductor_SMD:L_0805_2012Metric_Pad1.15x1.40mm_HandSolder
- R1, R2, R3, R4, R5, R6, R7: footprint (none) -> Resistor_SMD:R_0805_2012Metric_Pad1.20x1.40mm_HandSolder
- SW1: footprint (none) -> Button_Switch_THT:SW_PUSH_6mm_H4.3mm
- U4: footprint (none) -> RF_Module:HOPERF_RFM9XW_SMD
- Y1: footprint (none) -> Crystal:Crystal_SMD_HC49-SD_HandSoldering
- Y2: footprint (none) -> Crystal:Crystal_SMD_Abracon_ABS25-4Pin_8.0x3.8mm
Connections:
- net labels added: ANT
- wire segments 220 -> 225
- no-connect marks 14 -> 11
Other:
- note added: "PCB Antenna"
